File: nanao-ms9-29-power.sch (KiCad schematic (older format))
At the start: 128 parts, among them CN901 B2P3-VH, CN901W1 Conn_01x03_Male, CN902 Conn_01x05_Female, CN903 Degauss, J449 Jumper_NO_Small, J476 Jumper_NO_Small, J478 Jumper_NO_Small, J526 Jumper_NO_Small, Q901 2SK1531, Q902 2SC2412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

Commit message: Add files via upload
Unify the nanao.lib for using it for MS2930
Fix some minor errors in the schematic.
Parts:
- added CN951: Conn_01x02_Male, symbol Connector:Conn_01x02_Male
- added J525: Jumper_NO_Small, symbol nanao:jumper
- CN903: symbol nanao:Degauss -> nanao:COIL
- J449, J476, J478, J526: symbol Device:Jumper_NC_Small -> nanao:jumper
- R906: value 220K -> 100
- T901: symbol nanao:TR -> nanao:MS9_T901
Connections:
- net labels added: 15, r969+, r969-
- net labels removed: B+++
- wire segments 342 -> 349
Other:
- note added: "(3 Watts)"
- note added: "B+ adjust: \n76v at 15KHz (do it first)\n116v at 24KHz"
- note added: "Low/High plug\nshorts R968/R969"
- note added: "not populated circuitry\nswitches the 15/24\nB+ (shorten R953)\nQ951, ZD951,R951,\nR952, Q952,\nR956, R957"
- note added: "not populated fan\nconnector (Wire15)"
- moved on the sheet: C953, R968, R969, TP2

Commit message: Fixes R425, R457
Parts:
- added L902: NP, symbol Device:L
Connections:
- wire segments 349 -> 351
Other:
- note added: "ZD901 is\nnot populated\non my board"
- note added: "replaced\nby a wire"
- moved on the sheet: Q901
Changed lines of the file:
@@
 Sheet 2 2
 Title "NANAO MS9-29"
-Date "2025-09-30"
-Rev "1.2"
+Date "2025-11-17"
+Rev "1.3"
 Comp "Franck BOURDONNEC"
 Comment1 ""
@@
 L Device:Q_NMOS_GDS Q901
 U 1 1 6E3F1B8B
-P 2750 2300
-F 0 "Q901" H 2450 2450 50  0000 L CNN
-F 1 "2SK1531" H 2350 2350 50  0000 L CNN
-F 2 "" H 2950 2400 50  0001 C CNN
-F 3 "" H 2750 2300 50  0001 C CNN
-	1    2750 2300
+P 2750 2500
+F 0 "Q901" H 2450 2650 50  0000 L CNN
+F 1 "2SK1531" H 2350 2550 50  0000 L CNN
+F 2 "" H 2950 2600 50  0001 C CNN
+F 3 "" H 2750 2500 50  0001 C CNN
+	1    2750 2500
 	-1   0    0    -1
 $EndComp
 Wire Wire Line
-	2650 2100 2650 1950
+	2650 2300 2650 2250
 Connection ~ 2650 1950
 Wire Wire Line
@@
 $EndComp
 Wire Wire Line
-	2650 2500 2650 2800
-Wire Wire Line
 	2650 3150 2650 3400
 $Comp
@@
 Wire Wire Line
 	2850 2800 2650 2800
-Connection ~ 2650 2800
 Wire Wire Line
 	2650 2800 2650 2850
@@
 Connection ~ 3250 2800
 Wire Wire Line
-	2950 2300 3700 2300
+	3250 2300 3700 2300
 Wire Wire Line
 	3700 2300 3700 2600
@@
 U 1 1 717D015C
 P 4900 2800
-F 0 "Q903" H 4800 3000 50  0000 L CNN
+F 0 "Q903" H 4650 2900 50  0000 L CNN
 F 1 "2SC2412" V 4950 2300 50  0000 L CNN
 F 2 "" H 5100 2900 50  0001 C CNN
@@
 P 3600 4350
 F 0 "Q906" H 3300 4400 50  0000 L CNN
-F 1 "2SC2412" V 3650 3850 50  0000 L CNN
+F 1 "2SC2412" H 3250 4200 50  0000 L CNN
 F 2 "" H 3800 4450 50  0001 C CNN
 F 3 "" H 3600 4350 50  0001 C CNN
@@
 U 1 1 82EBCD07
 P 4550 2800
-F 0 "Q904" H 4450 3000 50  0000 L CNN
+F 0 "Q904" H 4300 2900 50  0000 L CNN
 F 1 "2SC2412" V 4600 2300 50  0000 L CNN
 F 2 "" H 4750 2900 50  0001 C CNN
@@
 Text Notes 1850 2250 0    24   ~ 0
 (3 Watts)
+Wire Wire Line
+	3250 2300 3250 2500
+Wire Wire Line
+	3250 2500 2950 2500
+Wire Wire Line
+	2650 2800 2650 2700
+Connection ~ 2650 2800
+$Comp
+L Device:L L902
+U 1 1 6927BF16
+P 2650 2100
+F 0 "L902" H 2700 2150 50  0000 L CNN
+F 1 "NP" H 2700 2050 50  0000 L CNN
+F 2 "" H 2650 2100 50  0001 C CNN
+F 3 "" H 2650 2100 50  0001 C CNN
+	1    2650 2100
+	1    0    0    -1
+$EndComp
+Text Notes 2900 2200 0    31   ~ 0
+replaced\nby a wire
+Text Notes 4300 1600 0    31   ~ 0
+ZD901 is\nnot populated\non my board
 $EndSCHEMATC

Commit message: Change F901 to 125v/6.3A(F)
Parts:
- F901: value 250v 3A -> 125v/6.3A(F)
Changed lines of the file:
@@
 Sheet 2 2
 Title "NANAO MS9-29"
-Date "2025-12-15"
-Rev "1.31"
+Date "2026-01-09"
+Rev "1.4"
 Comp "Franck BOURDONNEC"
 Comment1 ""
@@
 P 3500 5850
 F 0 "F901" V 3600 5850 50  0000 C CNN
-F 1 "250v 3A" V 3400 5900 50  0000 C CNN
+F 1 "125v/6.3A(F)" V 3400 5900 50  0000 C CNN
 F 2 "" V 3430 5850 50  0001 C CNN
 F 3 "" H 3500 5850 50  0001 C CNN
