File: nanao-ms9-29.sch (KiCad schematic (older format))
At the start: 506 parts, among them CN101 JST JH, CN101W1 Conn_01x06_Male, CN102 Conn_01x08_Male, CN280 Conn_01x12_Male, CN301 Conn_01x01_Male, CN301W1 Conn_01x01_Female, CN302 JST JH, CN303 Conn_01x05_Female, CN402 B10B_PH-K-S, CN570 Conn_01x05_Male, J281 Jumper_NO_Small, J282 Jumper_NO_Small, J283 Jumper_NO_Small, J284 Jumper_NO_Small, J293 33K, J307 Jumper_NO_Small, J401 Jumper_NO_Small, J404 Jumper_NO_Small, J409 Jumper_NO_Small, J411 Jumper_NO_Small, J419 1K, J430 Jumper_NO_Small, J433 6K8, J435 Jumper_NO_Small, J444 Jumper_NO_Small, J479 Jumper_NO_Small, J482 Jumper_NO_Small, J486 Jumper_NO_Small, J509 Jumper_NO_Small, J510 Jumper_NO_Small, J513 Jumper_NO_Small, J515 Jumper_NO_Small, J524 10K, Q101 2SC2412, Q102 2SC2412, Q201 2SA1037, Q202 2SA1037, Q203 2SA1037, Q204 2SC2412, Q205 2SA1037, Q301 2SC1740, Q302 2SC1044, Q303 2SC4218, Q304 2SA1624, Q311 2SC1740, Q312 2SC1044, Q313 2SC4218, Q314 2SA1624, Q321 2SC1740, Q322 2SC1044, Q323 2SC4218, Q324 2SA1624, Q401 2SC2412, Q402 2SC2412, Q403 2SD2400A, Q404 2SB1569A, Q451 2SA1037, Q452 DTC144E, Q501 2SC2412, Q502 2SA1037, Q503 2SA1020, Q506 2SC4692, Q507 2SK941, Q508 2SD1944, Q550 2SA1037, Q551 2SC2412, Q552 2SA1037, Q553 DTC143E, Q554 2SC2412, Q555 DTC144E, SW280 NP, T501 05F13617A1, T502 05F13618A1, U101 74LS86, U201 M51387P, U401 LA7837, U402 UPC358, U450 AN5551, U451 4558, U501 UPC358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

Commit message: Add files via upload
Unify the nanao.lib for using it for MS2930
Fix some minor errors in the schematic.
Parts:
- removed TP10, TP12, TP13, TP14, TP15, TP26, TP28, TP3, TP30, TP32, TP4, TP5, TP6, TP7, TP8, TP9: N, symbol nanao:TestPoint_Small
- added C204, C205, C206, C207, C208, C209: 100n, symbol Device:C
- added C4xx: 10n, symbol Device:C
- added CN503, CN504, CN505: Conn_01x04_Male, symbol Connector:Conn_01x04_Male
- added CN?: Conn_01x04_Female, symbol Connector:Conn_01x04_Female
- added J477, J483: Jumper_NO_Small, symbol nanao:jumper
- C411: value 2µ2 NoPola -> 2µ2 bipolar
- J281, J282, J283, J284, J307, J401, J409, J411, J430, J435, J444, J479, J482, J486, J509, J510, J513, J515: symbol Device:Jumper_NC_Small -> nanao:jumper
- T502: symbol nanao:EHT -> nanao:MS9_T502
- renumbered C508_or_C520 to C520, YOKE2 to DX1, YOKE1 to DY1
Connections:
- net labels added: r969+, r969-, wireD
- net labels removed: B+++
- wire segments 1345 -> 1387
Other:
- note added: "ASL, ABL, white field brighness adjustment\nOnly some jumpers are reported\nD, R and C are sometimes swapped when in serial.\nNP is not populated, although present on the original schematic\nSOT-23 diodes are used in paralell when only one is needed (eg pin 1 pin 2 linked)\nZD902 ZD903 to measure"
- note added: "B2P-VH"
- note added: "Not populated"
- note added: "PLUG+HIGH:\nC507 (1µ) S.Corr\nshort R968 R969 (higher B+)\nC506 serial with C504\nE1524=12v"
- note added: "PLUG+LOW:\nadd C519 to C507 (680n+1µ)\nunshort R968 R969\nshort C506\nE1524=0v"
- note added: "See https://mikejmoffitt.com/pages/ms9-hax/\nThis section improves sharpness by\nproviding a negative voltage to G1\nR517: 1K ,R518: 22K\nC521: 10µ 100v\nD506: sot23 (100v)\n"
- note added: "factory addition\nnear pin8 pin11 of ic401"
- note removed: "ASL, ABL, white field brighness adjustment\nOnly some jumpers are reported\nD, R and C are sometimes swapped when in serial.\nNP is not populated, although present on the original schematic\nSOT-23 diodes are used in paralell when only one is needed (eg pin 1 pin 2 linked)\nZD902 ZD903 undeterlined"
- note removed: "CN402 B2P-VH\nfor normal/miror"
- note removed: "CN503"
- note removed: "CN504"
- note removed: "CN505"
- note removed: "NP"
- note removed: "See https://mikejmoffitt.com/pages/ms9-hax/\nThis section improves sharpness by\nproviding a negative voltage to G1\nR517: 1K\nR518: 22K\nD506: sot23 (100v)\n"
- moved on the sheet: C504, C505, C506, C507, C520, CN301, CN301W1, L501, L504, R238, R467, R476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

Commit message: Add files via upload
Some fixes around hsize_adj not linked.
Use nanao.lib from ms2930
Parts:
- added C565: 100n, symbol Device:C
- added J111: 10K, symbol Device:R
- added J434: Jumper_NO_Small, symbol nanao:jumper
- D450: symbol Diode:1N4007 -> nanao:DANA202ALT
- renumbered R565 to R548
Connections:
- net labels added: ~E1524~
- net labels removed: EE1524, SPC1524
- wire segments 1387 -> 1396
Other:
- note removed: "R566 is strange"
- moved on the sheet: C410, C556, C557, C561, C566, Q451, Q452, Q552, Q553, Q555, R467, R469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

Commit message: Fixes R425, R457
Changed lines of the file:
@@
 Sheet 1 2
 Title "NANAO MS9-29"
-Date "2025-09-30"
-Rev "1.2"
+Date "2025-11-17"
+Rev "1.3"
 Comp "Franck BOURDONNEC"
 Comment1 ""
@@
 U 1 1 68E04A15
 P 9450 11200
-F 0 "Q401" H 9650 11200 50  0000 L CNN
-F 1 "2SC2412" H 9600 11100 50  0000 L CNN
+F 0 "Q401" H 9650 11250 50  0000 L CNN
+F 1 "2SC2412" H 9650 11150 50  0000 L CNN
 F 2 "" H 9650 11300 50  0001 C CNN
 F 3 "" H 9450 11200 50  0001 C CNN
@@
 U 1 1 7FF68640
 P 12600 12100
-F 0 "C409" H 12700 12100 50  0000 L CNN
-F 1 "120µ/35v" H 12700 12000 50  0000 L CNN
+F 0 "C409" H 12700 12150 50  0000 L CNN
+F 1 "120µ/35v" H 12700 12050 50  0000 L CNN
 F 2 "" H 12638 11950 50  0001 C CNN
 F 3 "" H 12600 12100 50  0001 C CNN
@@
 U 1 1 84F6CD8E
 P 16500 11850
-F 0 "C564" H 16600 11850 50  0000 L CNN
-F 1 "470n" H 16600 11950 50  0000 L CNN
+F 0 "C564" H 16600 11800 50  0000 L CNN
+F 1 "470n" H 16600 11900 50  0000 L CNN
 F 2 "" H 16538 11700 50  0001 C CNN
 F 3 "" H 16500 11850 50  0001 C CNN
@@
 U 1 1 7FDDB612
 P 11950 11250
-F 0 "Q403" H 12150 11250 50  0000 L CNN
-F 1 "2SD2400A" H 12150 11150 50  0000 L CNN
+F 0 "Q403" H 12150 11300 50  0000 L CNN
+F 1 "2SD2400A" H 12150 11200 50  0000 L CNN
 F 2 "" H 12150 11350 50  0001 C CNN
 F 3 "" H 11950 11250 50  0001 C CNN
@@
 Wire Bus Line
 	18650 4700 22800 4700
+Text Notes 8250 9450 2    24   ~ 0
+(fuse)
 $EndSCHEMATC

Commit message: minor comment on R457
Other:
- note added: "(sometimes incorrectly listed as 220K)"
Changed lines of the file:
@@
 	0    -1   -1   0
 $EndComp
-Text Notes 7900 12150 2    24   ~ 0
-(fuse)
+Text Notes 8500 12250 2    24   ~ 0
+(sometimes incorrectly listed as 220K)
 Text Notes 2350 14500 0    79   ~ 16
 H.POS
@@
 Wire Wire Line
 	12050 14900 12050 14950
+Text Notes 8250 9450 2    24   ~ 0
+(fuse)
+Text Notes 7900 12200 2    24   ~ 0
+(fuse)
 Wire Bus Line
 	22800 4700 22800 9250
 Wire Bus Line
 	18650 4700 22800 4700
-Text Notes 8250 9450 2    24   ~ 0
-(fuse)
 $EndSCHEMATC

Commit message: Add files via upload
minor warning about R532 value
Other:
- note added: "Check your board, service guide MS9-29SU \nsays 1R5 1/4watt lot of variation here !"
Changed lines of the file:
@@
 Sheet 1 2
 Title "NANAO MS9-29"
-Date "2025-11-17"
-Rev "1.3"
+Date "2025-12-15"
+Rev "1.31"
 Comp "Franck BOURDONNEC"
 Comment1 ""
@@
 Text Notes 7900 12200 2    24   ~ 0
 (fuse)
+Text Notes 20650 9500 0    31   ~ 0
+Check your board, service guide MS9-29SU \nsays 1R5 1/4watt lot of variation here !
 Wire Bus Line
 	22800 4700 22800 9250
